Commit message: updated sensor rig

File: ros2_ws/src/leap_desc/urdf/amiga_base.xacro (robot description, xacro)
@@ -1,5 +1,4 @@
 <?xml version="1.0" encoding="utf-8"?>
 <robot name="amiga_base" xmlns:xacro="http://www.ros.org/wiki/xacro">
-  <!-- base_link -->
   <link name="base_link">
     <inertial>
@@ -22,5 +21,4 @@
     </collision>
   </link>
-  <!-- base_footprint is used with Nav2 -->
   <link name="base_footprint" />
   <joint name="dummy_joint" type="fixed" >
@@ -28,5 +26,4 @@
     <child link="base_footprint" />
   </joint>
-  <!-- FL_wheel -->
   <link name="FL_wheel">
     <inertial>
@@ -55,5 +52,4 @@
     <axis xyz="0 0 1" />
   </joint>
-  <!-- FR_wheel -->
   <link name="FR_wheel">
     <inertial>
@@ -82,5 +78,4 @@
     <axis xyz="0 0 1" />
   </joint>
-  <!-- RL_wheel -->
   <link name="RL_wheel">
     <inertial>
@@ -109,5 +104,4 @@
     <axis xyz="0 0 1" />
   </joint>
-  <!-- RR_wheel -->
   <link name="RR_wheel">
     <inertial>
@@ -136,10 +130,66 @@
     <axis xyz="0 0 1" />
   </joint>
-  <!-- front_camera_hinge -->
-  <link name="front_camera_hinge">
-    <inertial>
-      <origin xyz="0.072808 -0.032484 -0.00017047" rpy="0 0 0" />
-      <mass value="0.21875" />
-      <inertia ixx="0.00029961" ixy="4.6954E-06" ixz="-3.6958E-07" iyy="0.00033063" iyz="2.5824E-07" izz="7.9946E-05" />
+  <joint name="slam_rig_mount_j" type="fixed">
+    <origin xyz="1.15 0.0 1.4" rpy="0 0 0" />
+    <parent link="base_link" />
+    <child link="slam_rig_base" />
+  </joint>
+  <link name="slam_rig_base">
+    <inertial>
+      <origin xyz="0.00050244 -1.1359E-06 0.030259" rpy="0 0 0" />
+      <mass value="0.45272" />
+      <inertia ixx="0.00025259" ixy="6.6853E-10" ixz="4.4531E-09" iyy="0.00024478" iyz="8.6751E-09" izz="0.00034312" />
+    </inertial>
+    <visual>
+      <origin xyz="0 0 0" rpy="0 0 0" />
+      <geometry>
+        <mesh filename="file://$(find leap_desc)/meshes/slam_rig_base.STL" />
+      </geometry>
+      <material name=""><color rgba="0.75294 0.75294 0.75294 1" /></material>
+    </visual>
+  </link>
+  <link name="os_sensor">
+    <inertial>
+      <origin xyz="-0.00086216 5.9592E-07 -0.034859" rpy="0 0 0" />
+      <mass value="0.83485" />
+      <inertia ixx="0.00063587" ixy="-1.6822E-07" ixz="-5.9486E-07" iyy="0.00063646" iyz="-1.1344E-08" izz="0.0010771" />
+    </inertial>
+    <visual>
+      <origin xyz="0 0 0" rpy="0 0 0" />
+      <geometry>
+        <mesh filename="file://$(find leap_desc)/meshes/ouster_lidar.STL" />
+      </geometry>
+      <material name=""><color rgba="0.79216 0.81961 0.93333 1" /></material>
+    </visual>
+  </link>
+  <joint name="ouster_lider_j" type="fixed">
+    <origin xyz="0 0 0.10803" rpy="0 0 0" />
+    <parent link="slam_rig_base" />
+    <child link="os_sensor" />
+  </joint>
+  <link name="RTK_gnss">
+    <inertial>
+      <origin xyz="8.6318E-08 1.3433E-08 -0.0064338" rpy="0 0 0" />
+      <mass value="0.046078" />
+      <inertia ixx="1.714E-05" ixy="-1.4122E-13" ixz="1.4571E-11" iyy="1.7117E-05" iyz="-4.7803E-12" izz="5.3861E-06" />
+    </inertial>
+    <visual>
+      <origin xyz="0 0 0" rpy="0 0 0" />
+      <geometry>
+        <mesh filename="file://$(find leap_desc)/meshes/RTK_gnss.STL"  />
+      </geometry>
+      <material name=""><color rgba="0.79216 0.81961 0.93333 1" /></material>
+    </visual>
+  </link>
+  <joint name="RTK_gnss_j" type="fixed">
+    <origin xyz="0 0 0.21003" rpy="0 0 0" />
+    <parent link="slam_rig_base" />
+    <child link="RTK_gnss" />
+  </joint>
+  <link name="camera">
+    <inertial>
+      <origin xyz="0.0013543 0.00036269 -0.00015622" rpy="0 0 0" />
+      <mass value="0.057213" />
+      <inertia ixx="5.9656E-06" ixy="4.8795E-08" ixz="5.2047E-08" iyy="9.9336E-06" iyz="-1.881E-08" izz="9.9952E-06" />
     </inertial>
     <visual>
@@ -148,52 +198,17 @@
         <mesh filename="file://$(find leap_desc)/meshes/camera.STL" />
       </geometry>
-      <material name=""><color rgba="1 0 0 1" /></material>
-    </visual>
-  </link>
-  <joint name="front_camera_hinge_j" type="fixed">
-    <origin xyz="1.1572 0.18502 1.1633" rpy="1.5708 -0.523599 0" />
-    <parent link="base_link" />
-    <child link="front_camera_hinge" />
-  </joint>
-  <!-- front_camera -->
-  <link name="front_camera"></link>
-  <joint name="front_camera_j" type="fixed">
-    <origin xyz="0.10238 -0.077341 0.0001016" rpy="-1.5708 0 -0.82903" />
-    <parent link="front_camera_hinge" />
-    <child link="front_camera" />
-  </joint>
-  <!-- front_camera_optical -->
-  <link name="front_camera_optical"></link>
-  <joint name="front_camera_optical_j" type="fixed">
+      <material name=""><color rgba="0.75294 0.75294 0.75294 1" /></material>
+    </visual>
+  </link>
+  <joint name="camera_j" type="fixed">
+    <origin xyz="0.049532 0 0.02659" rpy="0 0 0" />
+    <parent link="slam_rig_base" />
+    <child link="camera" />
+  </joint>
+  <link name="camera_optical" />
+  <joint name="camera_optical_j" type="fixed">
     <origin xyz="0 0 0" rpy="-1.5708 0 -1.5708" />
-    <parent link="front_camera" />
-    <child link="front_camera_optical" />
-  </joint>
-  <!-- lidar_hinge -->
-  <link name="lidar_hinge">
-    <inertial>
-      <origin xyz="0.12957 -0.043305 -0.00024862" rpy="0 0 0" />
-      <mass value="5.5092" />
-      <inertia ixx="0.0061651" ixy="0.0013206" ixz="-1.4672E-06" iyy="0.0076386" iyz="1.274E-06" izz="0.0071961" />
-    </inertial>
-    <visual>
-      <origin xyz="0 0 0" rpy="0 0 0" />
-      <geometry>
-        <mesh filename="file://$(find leap_desc)/meshes/lidar.STL" />
-      </geometry>
-      <material name=""><color rgba="0 1 0 1" /></material>
-    </visual>
-  </link>
-  <joint name="lidar_hinge_j" type="fixed">
-    <origin xyz="1.1572 0.18502 1.449" rpy="1.5708 -0.4363 0" />
-    <parent link="base_link" />
-    <child link="lidar_hinge" />
-  </joint>
-  <!-- lidar -->
-  <link name="lidar"></link>
-  <joint name="lidar_j" type="fixed">
-    <origin xyz="0.14354 -0.042185 0" rpy="-1.5708 0 -0.43633" />
-    <parent link="lidar_hinge" />
-    <child link="lidar" />
+    <parent link="camera" />
+    <child link="camera_optical" />
   </joint>
 </robot>

File: ros2_ws/src/leap_sim/urdf/amiga_sim.xacro (robot description, xacro)
@@ -3,13 +3,13 @@
   <!-- Import the pure hardware URDF -->
   <xacro:include filename="$(find leap_desc)/urdf/amiga_base.xacro" />
-  <!-- Gazebo Camera Sensor -->
-  <gazebo reference="front_camera">
+  <!-- Gazebo Camera Sensor: FLIR Blackfly S USB3 -->
+  <gazebo reference="camera">
     <sensor name="camera" type="camera">
       <camera>
         <camera_info_topic>camera/camera_info</camera_info_topic>
-        <horizontal_fov>1.047</horizontal_fov>
+        <horizontal_fov>1.5708</horizontal_fov>  <!-- this is 90 degrees, check against real sensor -->
         <image>
-          <width>320</width>
-          <height>240</height>
+          <width>1440</width>
+          <height>1080</height>
         </image>
         <clip>
@@ -22,9 +22,9 @@
       <visualize>true</visualize>
       <topic>camera/image_raw</topic>
-      <gz_frame_id>front_camera_optical</gz_frame_id>
+      <gz_frame_id>camera_optical</gz_frame_id>
     </sensor>
   </gazebo>
-  <!-- Gazebo LiDAR Sensor -->
-  <gazebo reference="lidar">
+  <!-- Gazebo LiDAR Sensor: Ouster OS0 Rev 7 -->
+  <gazebo reference="os_sensor">
     <sensor name='gpu_lidar' type='gpu_lidar'>
       <pose>0 0 0 0 0 0</pose>
@@ -33,37 +33,49 @@
       <ray>
         <scan>
+          <!-- OS0 True Horizontal: 360 degrees (2*pi) -->
           <horizontal>
-            <samples>640</samples>
+            <samples>1024</samples>
             <resolution>1</resolution>
-            <min_angle>-1.396263</min_angle>
-            <max_angle>1.396263</max_angle>
+            <min_angle>-3.14159</min_angle>
+            <max_angle>3.14159</max_angle>
           </horizontal>
+          <!-- OS0 True Vertical flattened to 1 layer for 2D Nav2 -->
           <vertical>
-            <samples>15</samples>
+            <samples>1</samples>
             <resolution>1</resolution>
-            <min_angle>-0.2618</min_angle>
-            <max_angle>0.2618</max_angle>
+            <min_angle>0.0</min_angle>
+            <max_angle>0.0</max_angle>
           </vertical>
         </scan>
         <range>
-          <min>0.08</min>
-          <max>10.0</max>
-          <resolution>0.01</resolution>
+          <min>0.1</min>
+          <max>35.0</max>
+          <resolution>0.003</resolution>
         </range>
       </ray>
       <always_on>1</always_on>
       <visualize>true</visualize>
-      <gz_frame_id>lidar</gz_frame_id>
+      <gz_frame_id>os_sensor</gz_frame_id>
     </sensor>
   </gazebo>
-  <!-- Untested IMU / GPS placeholders -->
-  <!--
-  <gazebo reference="imu">
-    <sensor name="imu_sensor" type="imu">... </sensor>
+  <!-- Gazebo IMU Sensor (Simulating the Ouster's internal IMU) -->
+  <gazebo reference="os_sensor">
+    <sensor name="imu_sensor" type="imu">
+      <always_on>true</always_on>
+      <update_rate>100</update_rate>
+      <visualize>true</visualize>
+      <topic>imu</topic>
+      <gz_frame_id>os_sensor</gz_frame_id>
+    </sensor>
   </gazebo>
-  <gazebo reference="gps">
-    <sensor name="navsat" type="navsat">... </sensor>
+  <!-- Gazebo GPS Sensor: Emlid Reach M2 -->
+  <gazebo reference="RTK_gnss">
+    <sensor name="reach_m2_navsat" type="navsat">
+      <always_on>true</always_on>
+      <update_rate>10</update_rate>
+      <topic>gps/fix</topic>
+      <gz_frame_id>RTK_gnss</gz_frame_id>
+    </sensor>
   </gazebo>
-  -->
   <!-- Gazebo ros2_control Hardware Interface -->
   <!-- Since the real robot uses a CAN black box, this is only needed in simulation -->

Commit message: refactored sensor code, updated urdf, added leap_launch, got localization mostly working

File: ros2_ws/src/leap_desc/urdf/amiga_base.xacro (robot description, xacro)
@@ -2,7 +2,7 @@
 <robot name="amiga_base" xmlns:xacro="http://www.ros.org/wiki/xacro">
   <link name="base_link">
-    <inertial>
-      <origin xyz="-0.054481 -0.015972 0.66252" rpy="0 0 0" />
-      <mass value="381.19" />
+    <inertial>  <!-- Guess -->
+      <origin xyz="0 0 0" rpy="0 0 0" />
+      <mass value="75" />
       <inertia ixx="5.717" ixy="-0.007109" ixz="0.0013622" iyy="12.857" iyz="1.2354E-05" izz="11.799" />
     </inertial>
@@ -10,5 +10,5 @@
       <origin xyz="0 0 0" rpy="0 0 0" />
       <geometry>
-        <mesh filename="file://$(find leap_desc)/meshes/frame_link.STL" />
+        <mesh filename="package://leap_desc/meshes/Frame.STL" />
       </geometry>
       <material name=""><color rgba="0.118 0.506 0.729 1" /></material>
@@ -17,5 +17,5 @@
       <origin xyz="0 0 0" rpy="0 0 0" />
       <geometry>
-        <mesh filename="file://$(find leap_desc)/meshes/frame_collision.STL"  />
+        <mesh filename="package://leap_desc/meshes/Frame.STL"  />
       </geometry>
     </collision>
@@ -26,188 +26,64 @@
     <child link="base_footprint" />
   </joint>
-  <link name="FL_wheel">
-    <inertial>
-      <origin xyz="4.3098E-07 5.5068E-07 -0.00020749" rpy="0 0 0" />
-      <mass value="15.628" />
-      <inertia ixx="0.153" ixy="1.1085E-06" ixz="2.7485E-07" iyy="0.153" iyz="2.341E-07" izz="0.28441" />
-    </inertial>
+  <link name="sensor_mount">
     <visual>
       <origin xyz="0 0 0" rpy="0 0 0" />
       <geometry>
-        <mesh filename="file://$(find leap_desc)/meshes/wheel.STL" />
-      </geometry>
-      <material name=""><color rgba="0 0 0 1" /></material>
-    </visual>
-    <collision>
-      <origin xyz="0 0 0" rpy="0 0 0" />
-      <geometry>
-        <mesh filename="file://$(find leap_desc)/meshes/wheel_collision.STL" />
-      </geometry>
-    </collision>
-  </link>
-  <joint name="FL_wheel_j" type="continuous">
-    <origin xyz="0.2658 0.32928 0.2159" rpy="1.5708 0 3.1416" />
-    <parent link="base_link" />
-    <child link="FL_wheel" />
-    <axis xyz="0 0 1" />
-  </joint>
-  <link name="FR_wheel">
-    <inertial>
-      <origin xyz="4.3153E-07 5.4433E-07 -0.00020748" rpy="0 0 0" />
-      <mass value="15.628" />
-      <inertia ixx="0.153" ixy="1.1081E-06" ixz="2.8146E-07" iyy="0.153" iyz="2.3106E-07" izz="0.28441" />
-    </inertial>
-    <visual>
-      <origin xyz="0 0 0" rpy="0 0 0" />
-      <geometry>
-        <mesh filename="file://$(find leap_desc)/meshes/wheel.STL" />
-      </geometry>
-      <material name=""><color rgba="0 0 0 1" /></material>
-    </visual>
-    <collision>
-      <origin xyz="0 0 0" rpy="0 0 0" />
-      <geometry>
-        <mesh filename="file://$(find leap_desc)/meshes/wheel_collision.STL" />
-      </geometry>
-    </collision>
-  </link>
-  <joint name="FR_wheel_j" type="continuous">
-    <origin xyz="0.2658 -0.32928 0.2159" rpy="1.5708 0 3.1416" />
-    <parent link="base_link" />
-    <child link="FR_wheel" />
-    <axis xyz="0 0 1" />
-  </joint>
-  <link name="RL_wheel">
-    <inertial>
-      <origin xyz="4.2324E-07 5.6831E-07 -0.00020749" rpy="0 0 0" />
-      <mass value="15.628" />
-      <inertia ixx="0.153" ixy="1.0985E-06" ixz="2.7036E-07" iyy="0.153" iyz="2.4709E-07" izz="0.28441" />
-    </inertial>
-    <visual>
-      <origin xyz="0 0 0" rpy="0 0 0" />
-      <geometry>
-        <mesh filename="file://$(find leap_desc)/meshes/wheel.STL" />
-      </geometry>
-      <material name=""><color rgba="0 0 0 1" /></material>
-    </visual>
-    <collision>
-      <origin xyz="0 0 0" rpy="0 0 0" />
-      <geometry>
-        <mesh filename="file://$(find leap_desc)/meshes/wheel_collision.STL" />
-      </geometry>
-    </collision>
-  </link>
-  <joint name="RL_wheel_j" type="continuous">
-    <origin xyz="-0.2658 0.32928 0.2159" rpy="1.5708 0 3.1416" />
-    <parent link="base_link" />
-    <child link="RL_wheel" />
-    <axis xyz="0 0 1" />
-  </joint>
-  <link name="RR_wheel">
-    <inertial>
-      <origin xyz="4.3464E-07 5.6185E-07 -0.00020748" rpy="0 0 0" />
-      <mass value="15.628" />
-      <inertia ixx="0.153" ixy="1.11E-06" ixz="2.6707E-07" iyy="0.153" iyz="2.4203E-07" izz="0.28441" />
-    </inertial>
-    <visual>
-      <origin xyz="0 0 0" rpy="0 0 0" />
-      <geometry>
-        <mesh filename="file://$(find leap_desc)/meshes/wheel.STL" />
-      </geometry>
-      <material name=""><color rgba="0 0 0 1" /></material>
-    </visual>
-    <collision>
-      <origin xyz="0 0 0" rpy="0 0 0" />
-      <geometry>
-        <mesh filename="file://$(find leap_desc)/meshes/wheel_collision.STL" />
-      </geometry>
-    </collision>
-  </link>
-  <joint name="RR_wheel_j" type="continuous">
-    <origin xyz="-0.2658 -0.32928 0.2159" rpy="1.5708 0 3.1416" />
-    <parent link="base_link" />
-    <child link="RR_wheel" />
-    <axis xyz="0 0 1" />
-  </joint>
-  <joint name="slam_rig_mount_j" type="fixed">
-    <origin xyz="1.15 0.0 1.4" rpy="0 0 0" />
-    <parent link="base_link" />
-    <child link="slam_rig_base" />
-  </joint>
-  <link name="slam_rig_base">
-    <inertial>
-      <origin xyz="0.00050244 -1.1359E-06 0.030259" rpy="0 0 0" />
-      <mass value="0.45272" />
-      <inertia ixx="0.00025259" ixy="6.6853E-10" ixz="4.4531E-09" iyy="0.00024478" iyz="8.6751E-09" izz="0.00034312" />
-    </inertial>
-    <visual>
-      <origin xyz="0 0 0" rpy="0 0 0" />
-      <geometry>
-        <mesh filename="file://$(find leap_desc)/meshes/slam_rig_base.STL" />
+        <mesh filename="package://leap_desc/meshes/SensorMount.STL" />
       </geometry>
       <material name=""><color rgba="0.75294 0.75294 0.75294 1" /></material>
     </visual>
   </link>
-  <link name="os_sensor">
-    <inertial>
-      <origin xyz="-0.00086216 5.9592E-07 -0.034859" rpy="0 0 0" />
-      <mass value="0.83485" />
-      <inertia ixx="0.00063587" ixy="-1.6822E-07" ixz="-5.9486E-07" iyy="0.00063646" iyz="-1.1344E-08" izz="0.0010771" />
-    </inertial>
+  <joint name="sensor_mount_j" type="fixed">
+    <origin xyz="-0.038587 0.0 0.340947" rpy="0 0 0" />
+    <parent link="base_link" />
+    <child link="sensor_mount" />
+  </joint>
+  <link name="ouster">
     <visual>
       <origin xyz="0 0 0" rpy="0 0 0" />
       <geometry>
-        <mesh filename="file://$(find leap_desc)/meshes/ouster_lidar.STL" />
+        <mesh filename="package://leap_desc/meshes/Ouster.STL" />
       </geometry>
       <material name=""><color rgba="0.79216 0.81961 0.93333 1" /></material>
     </visual>
   </link>
-  <joint name="ouster_lider_j" type="fixed">
-    <origin xyz="0 0 0.10803" rpy="0 0 0" />
-    <parent link="slam_rig_base" />
-    <child link="os_sensor" />
+  <joint name="ouster_j" type="fixed">
+    <origin xyz="0.000233 0 0.047625" rpy="0 0 0" />
+    <parent link="sensor_mount" />
+    <child link="ouster" />
   </joint>
-  <link name="RTK_gnss">
-    <inertial>
-      <origin xyz="8.6318E-08 1.3433E-08 -0.0064338" rpy="0 0 0" />
-      <mass value="0.046078" />
-      <inertia ixx="1.714E-05" ixy="-1.4122E-13" ixz="1.4571E-11" iyy="1.7117E-05" iyz="-4.7803E-12" izz="5.3861E-06" />
-    </inertial>
+  <link name="reach">
     <visual>
       <origin xyz="0 0 0" rpy="0 0 0" />
       <geometry>
-        <mesh filename="file://$(find leap_desc)/meshes/RTK_gnss.STL"  />
+        <mesh filename="package://leap_desc/meshes/Reach.STL"  />
       </geometry>
       <material name=""><color rgba="0.79216 0.81961 0.93333 1" /></material>
     </visual>
   </link>
-  <joint name="RTK_gnss_j" type="fixed">
-    <origin xyz="0 0 0.21003" rpy="0 0 0" />
-    <parent link="slam_rig_base" />
-    <child link="RTK_gnss" />
+  <joint name="reach_j" type="fixed">
+    <origin xyz="0.000233 0 0.148475" rpy="0 0 0" />
+    <parent link="sensor_mount" />
+    <child link="reach" />
   </joint>
-  <link name="camera">
-    <inertial>
-      <origin xyz="0.0013543 0.00036269 -0.00015622" rpy="0 0 0" />
-      <mass value="0.057213" />
-      <inertia ixx="5.9656E-06" ixy="4.8795E-08" ixz="5.2047E-08" iyy="9.9336E-06" iyz="-1.881E-08" izz="9.9952E-06" />
-    </inertial>
+  <link name="blackfly">
     <visual>
       <origin xyz="0 0 0" rpy="0 0 0" />
       <geometry>
-        <mesh filename="file://$(find leap_desc)/meshes/camera.STL" />
+        <mesh filename="package://leap_desc/meshes/Blackfly.STL" />
       </geometry>
       <material name=""><color rgba="0.75294 0.75294 0.75294 1" /></material>
     </visual>
   </link>
-  <joint name="camera_j" type="fixed">
-    <origin xyz="0.049532 0 0.02659" rpy="0 0 0" />
-    <parent link="slam_rig_base" />
-    <child link="camera" />
+  <joint name="blackfly_j" type="fixed">
+    <origin xyz="0.033516 0 0.012340" rpy="0 0 0" />
+    <parent link="sensor_mount" />
+    <child link="blackfly" />
   </joint>
   <link name="camera_optical" />
   <joint name="camera_optical_j" type="fixed">
     <origin xyz="0 0 0" rpy="-1.5708 0 -1.5708" />
-    <parent link="camera" />
+    <parent link="blackfly" />
     <child link="camera_optical" />
   </joint>

Commit message: urdf/tf bug fixing (still an issue that the sensor frames are arbitrary)

File: ros2_ws/src/leap_desc/urdf/amiga_base.xacro (robot description, xacro)
@@ -1,4 +1,5 @@
 <?xml version="1.0" encoding="utf-8"?>
 <robot name="amiga_base" xmlns:xacro="http://www.ros.org/wiki/xacro">
+  <link name="base_footprint"/>
   <link name="base_link">
     <inertial>  <!-- Guess -->
@@ -10,5 +11,5 @@
       <origin xyz="0 0 0" rpy="0 0 0" />
       <geometry>
-        <mesh filename="package://leap_desc/meshes/Frame.STL" />
+        <mesh filename="package://leap_desc/meshes/Frame.stl" />
       </geometry>
       <material name=""><color rgba="0.118 0.506 0.729 1" /></material>
@@ -17,12 +18,12 @@
       <origin xyz="0 0 0" rpy="0 0 0" />
       <geometry>
-        <mesh filename="package://leap_desc/meshes/Frame.STL"  />
+        <mesh filename="package://leap_desc/meshes/Frame.stl"  />
       </geometry>
     </collision>
   </link>
-  <link name="base_footprint" />
-  <joint name="dummy_joint" type="fixed" >
-    <parent link="base_link" />
-    <child link="base_footprint" />
+  <joint name="base_link_joint" type="fixed">
+    <parent link="base_footprint"/>
+    <child link="base_link"/>
+    <origin xyz="0 0 0.65" rpy="0 0 0"/>
   </joint>
   <link name="sensor_mount">
@@ -30,7 +31,7 @@
       <origin xyz="0 0 0" rpy="0 0 0" />
       <geometry>
-        <mesh filename="package://leap_desc/meshes/SensorMount.STL" />
+        <mesh filename="package://leap_desc/meshes/SensorMount.stl" />
       </geometry>
-      <material name=""><color rgba="0.75294 0.75294 0.75294 1" /></material>
+      <material name=""><color rgba="0.118 0.506 0.729 1" /></material>
     </visual>
   </link>
@@ -44,5 +45,5 @@
       <origin xyz="0 0 0" rpy="0 0 0" />
       <geometry>
-        <mesh filename="package://leap_desc/meshes/Ouster.STL" />
+        <mesh filename="package://leap_desc/meshes/Ouster.stl" />
       </geometry>
       <material name=""><color rgba="0.79216 0.81961 0.93333 1" /></material>
@@ -58,5 +59,5 @@
       <origin xyz="0 0 0" rpy="0 0 0" />
       <geometry>
-        <mesh filename="package://leap_desc/meshes/Reach.STL"  />
+        <mesh filename="package://leap_desc/meshes/Reach.stl"  />
       </geometry>
       <material name=""><color rgba="0.79216 0.81961 0.93333 1" /></material>
@@ -72,5 +73,5 @@
       <origin xyz="0 0 0" rpy="0 0 0" />
       <geometry>
-        <mesh filename="package://leap_desc/meshes/Blackfly.STL" />
+        <mesh filename="package://leap_desc/meshes/Blackfly.stl" />
       </geometry>
       <material name=""><color rgba="0.75294 0.75294 0.75294 1" /></material>

Commit message: updated urdf

File: ros2_ws/src/leap_desc/urdf/amiga_base.xacro (robot description, xacro)
@@ -51,5 +51,5 @@
   </link>
   <joint name="ouster_j" type="fixed">
-    <origin xyz="0.000233 0 0.047625" rpy="0 0 0" />
+    <origin xyz="0.000233 0 0.108065" rpy="0 0 0" />
     <parent link="sensor_mount" />
     <child link="ouster" />
@@ -83,9 +83,9 @@
     <child link="blackfly" />
   </joint>
-  <link name="camera_optical" />
-  <joint name="camera_optical_j" type="fixed">
+  <link name="blackfly_optical" />
+  <joint name="blackfly_optical_j" type="fixed">
     <origin xyz="0 0 0" rpy="-1.5708 0 -1.5708" />
     <parent link="blackfly" />
-    <child link="camera_optical" />
+    <child link="blackfly_optical" />
   </joint>
 </robot>

File: ros2_ws/src/leap_sim/urdf/amiga_sim copy.xacro (robot description, xacro)
@@ -22,5 +22,5 @@
       <visualize>true</visualize>
       <topic>camera/image_raw</topic>
-      <gz_frame_id>camera_optical</gz_frame_id>
+      <gz_frame_id>blackfly_optical</gz_frame_id>
     </sensor>
   </gazebo>

File: ros2_ws/src/leap_sim/urdf/amiga_sim.xacro (robot description, xacro)
@@ -22,5 +22,5 @@
       <visualize>true</visualize>
       <topic>camera/image_raw</topic>
-      <gz_frame_id>camera_optical</gz_frame_id>
+      <gz_frame_id>blackfly_optical</gz_frame_id>
     </sensor>
   </gazebo>
